File: Proto Business Card.brd (EAGLE design)
At the start: 50.8 x 88.9 mm, 579 parts

Commit message: Modified flower pads to shrink spacing, remove msak between pads, and shrink the via thickness. Added silk to the Arduino headers, and removed the K-Map text combinations in the back
Parts:
- U$170, U$575: value VIA.2-2.CORNER -> VIA.3-3; device flowerpad:2-2.CORNER -> flowerpad:3-3
- turned U$170 to 0 degrees
Routing:
- removed copper zone on layer 16, net N$119
- removed copper zone on layer 16, net N$120
- removed copper zone on layer 16, net N$121
- removed copper zone on layer 16, net N$122
Other:
- board text added: "v0.2"
- board text removed: "!C"
- board text removed: "!C!M"
- board text removed: "!C!S"
- board text removed: "!CM"
- board text removed: "!CS"
- board text removed: "!M"
- board text removed: "!M!S"
- board text removed: "!MS"
- board text removed: "!S"
- board text removed: "C"
- board text removed: "C!M"
- board text removed: "C!S"
- board text removed: "C!T"
- board text removed: "CM"
- board text removed: "CS"
- board text removed: "CT"
- board text removed: "M"
- board text removed: "M!S"
- board text removed: "M!T"
- board text removed: "MS"
- board text removed: "MT"
- board text removed: "S"
- board text removed: "S!T"
- board text removed: "ST"
